File: electronics/node.kicad_sch (KiCad schematic)
At the start: 43 parts

Commit message: working on stm32 debugging and accessory components
Parts:
- removed C?: 100pF, symbol Device:C
- removed C? (x2): 10uF, symbol Device:C
- removed C?: 0.01uF, symbol Device:C
- removed D?: D_Schottky, symbol Device:D_Schottky
- removed L?: CBC2518T100M, INDC2518X200N, symbol CBC2518T100M:CBC2518T100M
- removed R?: 274K, symbol Device:R
- removed R?: 10K, symbol Device:R
- removed R?: 100K, symbol Device:R
- removed R?: 1M, symbol Device:R
- removed U?: MIC2145BMM, symbol MIC2145BMM:MIC2145BMM
- added C? (x2): 10uF, symbol Device:C
- added C? (x2): 1uF, symbol Device:C
- added C?: 0.01uF, symbol Device:C
- added C?: 100pF, symbol Device:C
- added D?: SS34, DIOM7959X265N, symbol SS34:SS34
- added D?: D_Schottky, symbol Device:D_Schottky
- added J?: Conn_01x06, symbol Connector_Generic:Conn_01x06
- added J?: Conn_ST_STDC14, symbol Connector:Conn_ST_STDC14
- added L?: CBC2518T100M, INDC2518X200N, symbol CBC2518T100M:CBC2518T100M
- added R? (x8): 22, symbol Device:R
- added R?: 1M, symbol Device:R
- added R?: 100K, symbol Device:R
- added R?: 100, symbol Device:R
- added R? (x2): 4.7K, symbol Device:R
- added R?: 5K, symbol Device:R
- added R? (x2): 10K, symbol Device:R
- added R?: 50K, symbol Device:R
- added U?: MIC2145BMM, symbol MIC2145BMM:MIC2145BMM
- added U?: STM32L476MEYx, Package_CSP:ST_WLCSP-81_Die415, symbol MCU_ST_STM32L4:STM32L476MEYx
- added U?: LD39015M33R, Package_TO_SOT_SMD:SOT-23-5, symbol Regulator_Linear:LD39015M33R
Connections:
- net GND: now also C?.2, C?.2, C?.2, C?.2, J?.11 (GNDDetect), J?.3 (Pin_3), J?.5 (GND), J?.7 (GND), R?.1, R?.1, R?.1, R?.1, R?.1, U?.2 (GND), U?.4 (PGND), U?.8 (SGND)
- net SCL: now also R?.1, U?.A5 (PG14)
- net SDA: now also R?.1
- net VBAT: now also C?.1, C?.1, L?.1, R?.2, U?.1 (IN), U?.3 (EN), U?.6 (VDD)
- net +5V renamed +3.3V
- net +3.3V: now also C?.1, J?.3 (VCC), R?.2, R?.2, U?.5 (OUT)
- new net: J?.8 (JTDO/SWO), R?.1
- new net: C?.2, C?.2, R?.1, R?.2, U?.7 (FB)
- new net: D?.A, J?.1 (Pin_1), R?.2
- new net: J?.2 (Pin_2), R?.2
- new net: J?.4 (Pin_4), R?.2
- new net: J?.5 (Pin_5), R?.2
- new net: J?.6 (Pin_6), R?.2
- new net: D?.C, R?.1
- new net: J?.4 (JTMS/SWDIO), R?.1
- new net: D?.2 (A), L?.2, U?.5 (SW)
- new net: C?.1, U?.2 (SS)
- new net: R?.2, U?.3 (RSET)
- new net: J?.12 (~{RST}), R?.1
- new net: J?.6 (JCLK/SWCLK), R?.1
- new net +12V: C?.1, C?.1, D?.1 (K), R?.2
- new net 12V(EN): R?.2, U?.1 (En)
- new net AIN_1: R?.2
- new net JCLK/SWCLK: R?.1, R?.2
- new net JTDO/SWO: R?.1, R?.2
- new net JTMS/SWDIO: R?.1, R?.2
- new net NRST/RST: R?.1, R?.2
- no-connect marks 1 -> 5
Other:
- note added: "12V Step-Up Converter"
- note added: "150mA"
- note added: "3.3V Low-dropout Regulator"
- note added: "50 uA (Quiescent) 0.1V @ 100mA (Drop-out)"
- note added: "6-Pin Debugger"
- note added: "Put 12V(EN) high to enable a 12 V output"
- note added: "STDC14"
- note added: "SWD Connectors (for debugging)"
- note added: "V(out) = 12.0 V R2 = (1.08 x R1) / (V(out) - 1.08)"
- note removed: "V(out) = 5.0 V R2 = (1.08 x R1) / (V(out) - 1.08)"
- moved on the sheet: C?, D?, J?, JP?, L?, Q?, R?, U?
