File: electronics/coms-boards/lora/lora.kicad_sch (KiCad schematic)
At the start: 6 parts

Commit message: updated to re-align with master
Parts:
- C1: renamed from C?; footprint (none) -> Capacitor_SMD:C_0805_2012Metric
- J1: renamed from J?; footprint LINX_CONUFL001-SMD-T -> CONUFL001-SMD-T:LINX_CONUFL001-SMD-T
- R1, R2: renamed from R?; footprint (none) -> Resistor_SMD:R_0805_2012Metric
- U1: renamed from U?; footprint (none) -> RFM95W-915S2:XCVR_RFM95W-915S2
- gave numbers to parts that had none: 1
Connections:
- net +3.3V: now also J2.59 (F6)
- net GND: now also J2.61 (F7)
- net GPIO0: now also J2.47 (F0/!INT!); no longer J2.61 (F7)
- net GPIO1: now also J2.51 (F2/PWM); no longer J2.59 (F6)
- net GPIO2: now also J2.53 (F3); no longer J2.57 (F5)
- net GPIO4/RST: now also J2.57 (F5); no longer J2.53 (F3)
- no-connect marks 3 -> 26
Other:
- note added: "11th October 2022 (Harvey Bates)"
- note added: "Identifier Pins"
- note added: "LoRa to M.2 Connector"
