File: electronics/motherboard/motherboard-full/motherboard-full.kicad_sch (KiCad schematic)
At the start: 72 parts, among them J1 TBP02R2-381-02BE, J10 ST1W008S4AR1500, J11 MICROMOD_FUNCTION__MAIN, J12 TBP02R2-381-03BE, J13 TBP02R2-381-03BE, J14 TBP02R2-381-02BE, J2 Conn_01x04_Male, J3 USB4145-03-0230-C_REVA, J4 MICROMOD_-2222-C, J6 Conn_01x06_Female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

Commit message: realign with master branch before kangaroo board is split into seperate repo
Parts:
- BT1: footprint 1048:BAT_1048 -> BAT_1048
Connections:
- net GND: now also BT1.C1-, BT1.C2-, SW1.1, SW2.1; no longer BT1.C1, BT1.C2, SW1.2, SW2.2
Other:
- moved on the sheet: R4
Changed lines of the file:
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@@
   (junction (at 362.966 230.251) (diameter 0) (color 0 0 0 0)
   )
-  (junction (at 64.135 251.079) (diameter 0) (color 0 0 0 0)
+  (junction (at 62.23 251.079) (diameter 0) (color 0 0 0 0)
   )
   (junction (at 88.392 66.04) (diameter 0) (color 0 0 0 0)
@@
   (no_connect (at 65.278 141.986))
   (no_connect (at 65.278 131.826))
+  (no_connect (at 33.909 225.425))
   (no_connect (at 81.915 243.459))
   (no_connect (at 81.915 238.379))
@@
   (no_connect (at 81.915 235.839))
   (no_connect (at 46.482 225.552))
-  (no_connect (at 51.562 202.692))
-  (no_connect (at 33.909 202.565))
   (no_connect (at 28.829 225.425))
   (no_connect (at 81.915 212.979))
@@
   (no_connect (at 218.567 216.154))
   (no_connect (at 218.567 221.234))
+  (no_connect (at 51.562 225.552))
   (no_connect (at 81.915 256.159))
   (no_connect (at 81.915 258.699))
@@
     (stroke (width 0) (type default) (color 0 0 0 0))
   )
-  (wire (pts (xy 63.246 251.079) (xy 64.135 251.079))
+  (wire (pts (xy 61.341 251.079) (xy 62.23 251.079))
     (stroke (width 0) (type default) (color 0 0 0 0))
   )
@@
     (stroke (width 0) (type default) (color 0 0 0 0))
   )
-  (wire (pts (xy 64.135 251.079) (xy 81.915 251.079))
+  (wire (pts (xy 62.23 251.079) (xy 81.915 251.079))
     (stroke (width 0) (type default) (color 0 0 0 0))
   )
@@
     )
   )
-  (global_label "I2C_SDA" (shape input) (at 63.246 251.079 180) (fields_autoplaced)
+  (global_label "I2C_SDA" (shape input) (at 61.341 251.079 180) (fields_autoplaced)
     (effects (font (size 1.27 1.27)) (justify right))
-    (property "Intersheet References" "${INTERSHEET_REFS}" (id 0) (at 53.2129 251.1584 0)
+    (property "Intersheet References" "${INTERSHEET_REFS}" (id 0) (at 51.3079 251.1584 0)
       (effects (font (size 1.27 1.27)) (justify right) hide)
     )
@@
     (pin "1")
   )
-  (symbol (lib_id "Device:R") (at 64.135 247.269 0) (unit 1)
+  (symbol (lib_id "Device:R") (at 62.23 247.269 0) (unit 1)
     (in_bom yes) (on_board yes) (fields_autoplaced)
-    (property "Reference" "R4" (id 0) (at 65.913 246.4343 0)
+    (property "Reference" "R4" (id 0) (at 64.008 246.4343 0)
       (effects (font (size 1.27 1.27)) (justify left))
     )
-    (property "Value" "4.7K" (id 1) (at 65.913 248.9712 0)
+    (property "Value" "4.7K" (id 1) (at 64.008 248.9712 0)
       (effects (font (size 1.27 1.27)) (justify left))
     )
-    (property "Footprint" "Resistor_SMD:R_0805_2012Metric" (id 2) (at 62.357 247.269 90)
+    (property "Footprint" "Resistor_SMD:R_0805_2012Metric" (id 2) (at 60.452 247.269 90)
       (effects (font (size 1.27 1.27)) hide)
     )
-    (property "Datasheet" "~" (id 3) (at 64.135 247.269 0)
+    (property "Datasheet" "~" (id 3) (at 62.23 247.269 0)
       (effects (font (size 1.27 1.27)) hide)
     )
@@
     (pin "1")
   )
-  (symbol (lib_id "power:GND") (at 33.909 225.425 0) (unit 1)
+  (symbol (lib_id "power:GND") (at 33.909 202.565 180) (unit 1)
     (in_bom yes) (on_board yes) (fields_autoplaced)
-    (property "Reference" "#PWR02" (id 0) (at 33.909 231.775 0)
+    (property "Reference" "#PWR02" (id 0) (at 33.909 196.215 0)
       (effects (font (size 1.27 1.27)) hide)
     )
-    (property "Value" "GND" (id 1) (at 33.909 229.8684 0))
-    (property "Footprint" "" (id 2) (at 33.909 225.425 0)
+    (property "Value" "GND" (id 1) (at 33.909 198.9892 0))
+    (property "Footprint" "" (id 2) (at 33.909 202.565 0)
       (effects (font (size 1.27 1.27)) hide)
     )
-    (property "Datasheet" "" (id 3) (at 33.909 225.425 0)
+    (property "Datasheet" "" (id 3) (at 33.909 202.565 0)
       (effects (font (size 1.27 1.27)) hide)
     )
@@
   (symbol (lib_id "power:GND") (at 65.278 154.686 90) (unit 1)
     (in_bom yes) (on_board yes)
-    (property "Reference" "#PWR?" (id 0) (at 71.628 154.686 0)
+    (property "Reference" "#PWR0101" (id 0) (at 71.628 154.686 0)
       (effects (font (size 1.27 1.27)) hide)
     )
@@
     (pin "1")
   )
-  (symbol (lib_id "power:+3.3V") (at 64.135 243.459 0) (unit 1)
+  (symbol (lib_id "power:+3.3V") (at 62.23 243.459 0) (unit 1)
     (in_bom yes) (on_board yes)
-    (property "Reference" "#PWR010" (id 0) (at 64.135 247.269 0)
+    (property "Reference" "#PWR010" (id 0) (at 62.23 247.269 0)
       (effects (font (size 1.27 1.27)) hide)
     )
-    (property "Value" "+3.3V" (id 1) (at 65.405 241.935 0)
+    (property "Value" "+3.3V" (id 1) (at 63.5 241.935 0)
       (effects (font (size 1.27 1.27)) (justify left))
     )
-    (property "Footprint" "" (id 2) (at 64.135 243.459 0)
+    (property "Footprint" "" (id 2) (at 62.23 243.459 0)
       (effects (font (size 1.27 1.27)) hide)
     )
-    (property "Datasheet" "" (id 3) (at 64.135 243.459 0)
+    (property "Datasheet" "" (id 3) (at 62.23 243.459 0)
       (effects (font (size 1.27 1.27)) hide)
     )
@@
     (pin "5")
   )
-  (symbol (lib_id "power:GND") (at 51.562 225.552 0) (unit 1)
+  (symbol (lib_id "power:GND") (at 51.562 202.692 180) (unit 1)
     (in_bom yes) (on_board yes) (fields_autoplaced)
-    (property "Reference" "#PWR06" (id 0) (at 51.562 231.902 0)
+    (property "Reference" "#PWR06" (id 0) (at 51.562 196.342 0)
       (effects (font (size 1.27 1.27)) hide)
     )
-    (property "Value" "GND" (id 1) (at 51.562 229.9954 0))
-    (property "Footprint" "" (id 2) (at 51.562 225.552 0)
+    (property "Value" "GND" (id 1) (at 51.562 199.1162 0))
+    (property "Footprint" "" (id 2) (at 51.562 202.692 0)
       (effects (font (size 1.27 1.27)) hide)
     )
-    (property "Datasheet" "" (id 3) (at 51.562 225.552 0)
+    (property "Datasheet" "" (id 3) (at 51.562 202.692 0)
       (effects (font (size 1.27 1.27)) hide)
     )
@@
       (effects (font (size 1.27 1.27)) (justify right))
     )
-    (property "Footprint" "1048:BAT_1048" (id 2) (at 347.98 29.718 0)
+    (property "Footprint" "BAT_1048" (id 2) (at 347.98 29.718 0)
       (effects (font (size 1.27 1.27)) (justify left bottom) hide)
     )
@@
       (effects (font (size 1.27 1.27)) (justify left bottom) hide)
     )
-    (pin "C1")
     (pin "C1+")
-    (pin "C2")
+    (pin "C1-")
     (pin "C2+")
+    (pin "C2-")
   )
   (symbol (lib_id "9774025151R:9774025151R") (at 183.642 128.016 0) (unit 1)
@@
     )
     (path "/37c1703b-3579-4596-bbc9-e3529b05bc7e"
-      (reference "#PWR?") (unit 1) (value "GND") (footprint "")
+      (reference "#PWR0101") (unit 1) (value "GND") (footprint "")
     )
     (path "/b1aa4c51-3236-44e8-aa45-cd71871f300e"
-      (reference "BT1") (unit 1) (value "1048") (footprint "1048:BAT_1048")
+      (reference "BT1") (unit 1) (value "1048") (footprint "BAT_1048")
     )
     (path "/295680e7-b94b-47e0-902b-5b0b1f42daea"
