File: electronics/breakout/breakout.kicad_pcb (KiCad board)
At the start: 2 copper layers, 114 x 146 mm, 55 parts, among them J1 2604-3103, J2 2604-3103, J3 2604-3103, J4 2604-3103, J5 2604-3103, J6 2604-3103, J7 2604-3103, J8 2604-3105, J9 2604-3103

Commit message: Breakout board main connector now in same order as on the Wombat board.
Parts:
- added REF**: small_nsw_gov, DPI:small_nsw_gov, F.Cu at (51.1, 100.5)
- moved kibuzzard-637324AF 20.0 mm to (105.2, 110.5)
- moved kibuzzard-6373244B 10.0 mm to (104.4, 105.5)
- moved kibuzzard-637323EC 10.0 mm to (105.1, 95.5)
- moved kibuzzard-63732487 10.0 mm to (104.1, 90.5)
- moved kibuzzard-637324B6 10.0 mm to (105.2, 100.5)
Connections:
- J8 pad 1: +12V -> +3.3V
- J8 pad 10: +3.3V -> Digital_Interrupt
- J8 pad 2: +12V -> +3.3V
- J8 pad 3: GND -> SDI-12_DATA
- J8 pad 4: GND -> SDI-12_DATA
- J8 pad 5: Digital_Interrupt -> +12V
- J8 pad 6: Digital_Interrupt -> +12V
- J8 pad 7: SDI-12_DATA -> GND
- J8 pad 8: SDI-12_DATA -> GND
- J8 pad 9: +3.3V -> Digital_Interrupt
Routing:
- net SDI-12_DATA: track 274.0 -> 282.5 mm
- net +12V: track 269.9 -> 277.9 mm
- net Digital_Interrupt: track 65.1 -> 61.0 mm
- net +3.3V: track 101.2 -> 98.1 mm
Other:
- board text removed: "Harvey Bates Nov 2022"
